Commit message: fix foot position of xacro

File: ros2_ws/src/biped_description/urdf/biped_digitigrade.urdf.xacro (robot description, xacro)
@@ -177,7 +177,8 @@
     </joint>
     <link name="${side}_foot_link">
-      <!-- 逆関節の足部: 後方（-X方向）に伸びる -->
-      <visual>
-        <origin xyz="${-foot_length/2} 0 ${-foot_height/2}" rpy="0 0 0"/>
+      <!-- 足首関節が足部の中心に位置する -->
+      <!-- 足部は前後に均等に広がる（前方 +X、後方 -X） -->
+      <visual>
+        <origin xyz="0 0 ${-foot_height/2}" rpy="0 0 0"/>
         <geometry>
           <box size="${foot_length} ${foot_width} ${foot_height}"/>
@@ -186,5 +187,5 @@
       </visual>
       <collision>
-        <origin xyz="${-foot_length/2} 0 ${-foot_height/2}" rpy="0 0 0"/>
+        <origin xyz="0 0 ${-foot_height/2}" rpy="0 0 0"/>
         <geometry>
           <box size="${foot_length} ${foot_width} ${foot_height}"/>
@@ -193,5 +194,5 @@
       <inertial>
         <mass value="0.3"/>
-        <origin xyz="${-foot_length/2} 0 ${-foot_height/2}" rpy="0 0 0"/>
+        <origin xyz="0 0 ${-foot_height/2}" rpy="0 0 0"/>
         <inertia ixx="0.001" ixy="0" ixz="0" iyy="0.001" iyz="0" izz="0.001"/>
       </inertial>

Commit message: add 3d model for rl

File: ros2_ws/src/biped_description/urdf/biped_digitigrade.urdf.xacro (robot description, xacro)
@@ -7,4 +7,5 @@
     - 片脚5関節 × 2脚（左右対称）
     - 関節構成: 腰ヨー, 股関節ロール, 股関節ピッチ, 膝ピッチ, 足首ピッチ
+    - IMUリンク: 胴体上面中央に配置（強化学習・状態推定用）
   -->
   <!-- リンク長パラメータ (example_gait.pyと一致) -->
@@ -55,4 +56,31 @@
     </inertial>
   </link>
+  <!-- IMU Link -->
+  <!--
+    IMUセンサの取り付け位置を定義するフレーム
+    - URDFではリンク+固定ジョイントとして定義（ROS 2標準）
+    - MuJoCo変換時にはsiteとして扱われ、gyro/accelerometer等のセンサを配置可能
+    - 質量・慣性は無視できる程度の小さい値（シミュレーションに影響しない）
+  -->
+  <link name="imu_link">
+    <visual>
+      <origin xyz="0 0 0" rpy="0 0 0"/>
+      <geometry>
+        <box size="0.02 0.02 0.01"/>
+      </geometry>
+      <material name="dark_gray"/>
+    </visual>
+    <inertial>
+      <mass value="0.01"/>
+      <origin xyz="0 0 0" rpy="0 0 0"/>
+      <inertia ixx="1e-6" ixy="0" ixz="0" iyy="1e-6" iyz="0" izz="1e-6"/>
+    </inertial>
+  </link>
+  <joint name="imu_joint" type="fixed">
+    <parent link="base_link"/>
+    <child link="imu_link"/>
+    <!-- IMUは胴体上面中央に配置 -->
+    <origin xyz="0 0 0.06" rpy="0 0 0"/>
+  </joint>
   <!-- 脚マクロ定義 -->
   <xacro:macro name="leg" params="side reflect">

Commit message: Revert "Feat/update rl walking -001(#7)"
This reverts commit 8a2bc420a66bb8beb061c2bfdad12e29c53db8d3.

File: ros2_ws/src/biped_description/urdf/biped_digitigrade.urdf.xacro (robot description, xacro)
@@ -7,5 +7,4 @@
     - 片脚5関節 × 2脚（左右対称）
     - 関節構成: 腰ヨー, 股関節ロール, 股関節ピッチ, 膝ピッチ, 足首ピッチ
-    - IMUリンク: 胴体上面中央に配置（強化学習・状態推定用）
   -->
   <!-- リンク長パラメータ (example_gait.pyと一致) -->
@@ -56,31 +55,4 @@
     </inertial>
   </link>
-  <!-- IMU Link -->
-  <!--
-    IMUセンサの取り付け位置を定義するフレーム
-    - URDFではリンク+固定ジョイントとして定義（ROS 2標準）
-    - MuJoCo変換時にはsiteとして扱われ、gyro/accelerometer等のセンサを配置可能
-    - 質量・慣性は無視できる程度の小さい値（シミュレーションに影響しない）
-  -->
-  <link name="imu_link">
-    <visual>
-      <origin xyz="0 0 0" rpy="0 0 0"/>
-      <geometry>
-        <box size="0.02 0.02 0.01"/>
-      </geometry>
-      <material name="dark_gray"/>
-    </visual>
-    <inertial>
-      <mass value="0.01"/>
-      <origin xyz="0 0 0" rpy="0 0 0"/>
-      <inertia ixx="1e-6" ixy="0" ixz="0" iyy="1e-6" iyz="0" izz="1e-6"/>
-    </inertial>
-  </link>
-  <joint name="imu_joint" type="fixed">
-    <parent link="base_link"/>
-    <child link="imu_link"/>
-    <!-- IMUは胴体上面中央に配置 -->
-    <origin xyz="0 0 0.06" rpy="0 0 0"/>
-  </joint>
   <!-- 脚マクロ定義 -->
   <xacro:macro name="leg" params="side reflect">
