Commit message: (WIP) updating robstride_hardware

File: ros2_ws/src/robstride_hardware/urdf/robstride_system.urdf.xacro (robot description, xacro)
@@ -1,5 +1,23 @@
 <?xml version="1.0"?>
 <robot xmlns:xacro="http://www.ros.org/wiki/xacro" name="robstride_robot">
-  <!-- Minimal robot description -->
+  <!-- ================================================================== -->
+  <!-- Xacro macro for a RobStride motor joint (ros2_control definition)  -->
+  <!-- ================================================================== -->
+  <xacro:macro name="robstride_joint" params="name can_interface motor_id kp kd">
+    <joint name="${name}">
+      <param name="can_interface">${can_interface}</param>
+      <param name="motor_id">${motor_id}</param>
+      <param name="kp">${kp}</param>
+      <param name="kd">${kd}</param>
+      <command_interface name="position"/>
+      <state_interface name="position"/>
+      <state_interface name="velocity"/>
+      <state_interface name="effort"/>
+    </joint>
+  </xacro:macro>
+  <!-- ================================================================== -->
+  <!-- Minimal robot description (dummy links for standalone testing)     -->
+  <!-- For the full model, use biped_description/urdf instead.            -->
+  <!-- ================================================================== -->
   <link name="base_link">
     <visual>
@@ -9,40 +27,29 @@
     </visual>
   </link>
-  <link name="joint1_link">
-    <visual>
-      <geometry>
-        <cylinder length="0.2" radius="0.05"/>
-      </geometry>
-    </visual>
-  </link>
-  <joint name="joint1" type="revolute">
+  <!-- Dummy link and fixed joint so URDF is valid with no movable joints -->
+  <link name="dummy_link"/>
+  <joint name="dummy_fixed" type="fixed">
     <parent link="base_link"/>
-    <child link="joint1_link"/>
-    <origin xyz="0 0 0.1" rpy="0 0 0"/>
-    <axis xyz="0 0 1"/>
-    <limit lower="-3.14" upper="3.14" effort="10.0" velocity="5.0"/>
+    <child link="dummy_link"/>
   </joint>
-  <!-- ros2_control configuration -->
+  <!-- ================================================================== -->
+  <!-- ros2_control configuration: 10 joints on 2 CAN buses              -->
+  <!-- ================================================================== -->
   <ros2_control name="robstride_system" type="system">
     <hardware>
       <plugin>robstride_hardware/RobStrideHardware</plugin>
-      <param name="can_interface">can1</param>
-      <param name="motor_id">127</param>
-      <param name="kp">1.5</param>
-      <param name="kd">0.01</param>
-      <!-- State reader thread configuration (200Hz, separate from RT loop) -->
-      <param name="state_reader_rate">200</param>
-      <param name="state_reader_cpu_affinity">3</param>
-      <param name="state_reader_priority">80</param>
     </hardware>
-    <joint name="joint1">
-      <command_interface name="position">
-        <param name="min">-3.14</param>
-        <param name="max">3.14</param>
-      </command_interface>
-      <state_interface name="position"/>
-      <state_interface name="velocity"/>
-      <state_interface name="effort"/>
-    </joint>
+    <!-- Left leg (CAN1) -->
+    <xacro:robstride_joint name="left_hip_yaw_joint"     can_interface="can1" motor_id="11" kp="30.0" kd="1.0"/>
+    <xacro:robstride_joint name="left_hip_roll_joint"    can_interface="can1" motor_id="12" kp="30.0" kd="1.0"/>
+    <xacro:robstride_joint name="left_hip_pitch_joint"   can_interface="can1" motor_id="13" kp="30.0" kd="1.0"/>
+    <xacro:robstride_joint name="left_knee_pitch_joint"  can_interface="can1" motor_id="14" kp="30.0" kd="1.0"/>
+    <xacro:robstride_joint name="left_ankle_pitch_joint" can_interface="can1" motor_id="15" kp="30.0" kd="1.0"/>
+    <!-- Right leg (CAN2) -->
+    <xacro:robstride_joint name="right_hip_yaw_joint"     can_interface="can2" motor_id="21" kp="30.0" kd="1.0"/>
+    <xacro:robstride_joint name="right_hip_roll_joint"    can_interface="can2" motor_id="22" kp="30.0" kd="1.0"/>
+    <xacro:robstride_joint name="right_hip_pitch_joint"   can_interface="can2" motor_id="23" kp="30.0" kd="1.0"/>
+    <xacro:robstride_joint name="right_knee_pitch_joint"  can_interface="can2" motor_id="24" kp="30.0" kd="1.0"/>
+    <xacro:robstride_joint name="right_ankle_pitch_joint" can_interface="can2" motor_id="25" kp="30.0" kd="1.0"/>
   </ros2_control>
 </robot>
