Commit message: rename in package dir

File: ros2_ws/src/aoba_hardware/urdf/aoba_system.urdf.xacro (robot description, xacro)
@@ -1,8 +1,8 @@
 <?xml version="1.0"?>
-<robot xmlns:xacro="http://www.ros.org/wiki/xacro" name="robstride_robot">
+<robot xmlns:xacro="http://www.ros.org/wiki/xacro" name="aoba_robot">
   <!-- ================================================================== -->
   <!-- Xacro macro for a RobStride motor joint (ros2_control definition)  -->
   <!-- ================================================================== -->
-  <xacro:macro name="robstride_joint" params="name can_interface motor_id kp kd">
+  <xacro:macro name="aoba_joint" params="name can_interface motor_id kp kd">
     <joint name="${name}">
       <param name="can_interface">${can_interface}</param>
@@ -36,20 +36,20 @@
   <!-- ros2_control configuration: 10 joints on 2 CAN buses              -->
   <!-- ================================================================== -->
-  <ros2_control name="robstride_system" type="system">
+  <ros2_control name="aoba_system" type="system">
     <hardware>
-      <plugin>robstride_hardware/RobStrideHardware</plugin>
+      <plugin>aoba_hardware/AobaHardware</plugin>
     </hardware>
     <!-- Left leg (CAN1) -->
-    <xacro:robstride_joint name="left_hip_yaw_joint"     can_interface="can1" motor_id="11" kp="30.0" kd="1.0"/>
-    <xacro:robstride_joint name="left_hip_roll_joint"    can_interface="can1" motor_id="12" kp="30.0" kd="1.0"/>
-    <xacro:robstride_joint name="left_hip_pitch_joint"   can_interface="can1" motor_id="13" kp="30.0" kd="1.0"/>
-    <xacro:robstride_joint name="left_knee_pitch_joint"  can_interface="can1" motor_id="14" kp="30.0" kd="1.0"/>
-    <xacro:robstride_joint name="left_ankle_pitch_joint" can_interface="can1" motor_id="15" kp="30.0" kd="1.0"/>
+    <xacro:aoba_joint name="left_hip_yaw_joint"     can_interface="can1" motor_id="11" kp="30.0" kd="1.0"/>
+    <xacro:aoba_joint name="left_hip_roll_joint"    can_interface="can1" motor_id="12" kp="30.0" kd="1.0"/>
+    <xacro:aoba_joint name="left_hip_pitch_joint"   can_interface="can1" motor_id="13" kp="30.0" kd="1.0"/>
+    <xacro:aoba_joint name="left_knee_pitch_joint"  can_interface="can1" motor_id="14" kp="30.0" kd="1.0"/>
+    <xacro:aoba_joint name="left_ankle_pitch_joint" can_interface="can1" motor_id="15" kp="30.0" kd="1.0"/>
     <!-- Right leg (CAN2) -->
-    <xacro:robstride_joint name="right_hip_yaw_joint"     can_interface="can2" motor_id="21" kp="30.0" kd="1.0"/>
-    <xacro:robstride_joint name="right_hip_roll_joint"    can_interface="can2" motor_id="22" kp="30.0" kd="1.0"/>
-    <xacro:robstride_joint name="right_hip_pitch_joint"   can_interface="can2" motor_id="23" kp="30.0" kd="1.0"/>
-    <xacro:robstride_joint name="right_knee_pitch_joint"  can_interface="can2" motor_id="24" kp="30.0" kd="1.0"/>
-    <xacro:robstride_joint name="right_ankle_pitch_joint" can_interface="can2" motor_id="25" kp="30.0" kd="1.0"/>
+    <xacro:aoba_joint name="right_hip_yaw_joint"     can_interface="can2" motor_id="21" kp="30.0" kd="1.0"/>
+    <xacro:aoba_joint name="right_hip_roll_joint"    can_interface="can2" motor_id="22" kp="30.0" kd="1.0"/>
+    <xacro:aoba_joint name="right_hip_pitch_joint"   can_interface="can2" motor_id="23" kp="30.0" kd="1.0"/>
+    <xacro:aoba_joint name="right_knee_pitch_joint"  can_interface="can2" motor_id="24" kp="30.0" kd="1.0"/>
+    <xacro:aoba_joint name="right_ankle_pitch_joint" can_interface="can2" motor_id="25" kp="30.0" kd="1.0"/>
   </ros2_control>
 </robot>

File: ros2_ws/src/aoba_hardware/urdf/single_motor_test.urdf.xacro (robot description, xacro)
@@ -1,4 +1,4 @@
 <?xml version="1.0"?>
-<robot xmlns:xacro="http://www.ros.org/wiki/xacro" name="robstride_single_motor_test">
+<robot xmlns:xacro="http://www.ros.org/wiki/xacro" name="aoba_single_motor_test">
   <!-- ================================================================== -->
   <!-- Single motor test configuration                                    -->
@@ -28,7 +28,7 @@
   </joint>
   <!-- ros2_control: single motor on can0 -->
-  <ros2_control name="robstride_system" type="system">
+  <ros2_control name="aoba_system" type="system">
     <hardware>
-      <plugin>robstride_hardware/RobStrideHardware</plugin>
+      <plugin>aoba_hardware/AobaHardware</plugin>
     </hardware>
     <joint name="test_joint">

Commit message: URDFで定めた回転方向と実際のモータの回転方向の符号を整合させるパラメータを追加

File: ros2_ws/src/aoba_hardware/urdf/aoba_system.urdf.xacro (robot description, xacro)
@@ -4,5 +4,5 @@
   <!-- Xacro macro for a RobStride motor joint (ros2_control definition)  -->
   <!-- ================================================================== -->
-  <xacro:macro name="aoba_joint" params="name can_interface motor_id kp kd">
+  <xacro:macro name="aoba_joint" params="name can_interface motor_id kp kd direction">
     <joint name="${name}">
       <param name="can_interface">${can_interface}</param>
@@ -10,4 +10,5 @@
       <param name="kp">${kp}</param>
       <param name="kd">${kd}</param>
+      <param name="direction">${direction}</param>
       <command_interface name="position"/>
       <state_interface name="position"/>
@@ -28,15 +29,15 @@
     </hardware>
     <!-- Left leg (CAN1) -->
-    <xacro:aoba_joint name="rev11" can_interface="can1" motor_id="11" kp="30.0" kd="1.0"/>
-    <xacro:aoba_joint name="rev12" can_interface="can1" motor_id="12" kp="30.0" kd="1.0"/>
-    <xacro:aoba_joint name="rev13" can_interface="can1" motor_id="13" kp="30.0" kd="1.0"/>
-    <xacro:aoba_joint name="rev14" can_interface="can1" motor_id="14" kp="30.0" kd="1.0"/>
-    <xacro:aoba_joint name="rev15" can_interface="can1" motor_id="15" kp="30.0" kd="1.0"/>
+    <xacro:aoba_joint name="rev11" can_interface="can1" motor_id="11" kp="30.0" kd="1.0" direction="-1"/>
+    <xacro:aoba_joint name="rev12" can_interface="can1" motor_id="12" kp="30.0" kd="1.0" direction="1"/>
+    <xacro:aoba_joint name="rev13" can_interface="can1" motor_id="13" kp="30.0" kd="1.0" direction="1"/>
+    <xacro:aoba_joint name="rev14" can_interface="can1" motor_id="14" kp="30.0" kd="1.0" direction="1"/>
+    <xacro:aoba_joint name="rev15" can_interface="can1" motor_id="15" kp="30.0" kd="1.0" direction="1"/>
     <!-- Right leg (CAN2) -->
-    <xacro:aoba_joint name="rev21" can_interface="can2" motor_id="21" kp="30.0" kd="1.0"/>
-    <xacro:aoba_joint name="rev22" can_interface="can2" motor_id="22" kp="30.0" kd="1.0"/>
-    <xacro:aoba_joint name="rev23" can_interface="can2" motor_id="23" kp="30.0" kd="1.0"/>
-    <xacro:aoba_joint name="rev24" can_interface="can2" motor_id="24" kp="30.0" kd="1.0"/>
-    <xacro:aoba_joint name="rev25" can_interface="can2" motor_id="25" kp="30.0" kd="1.0"/>
+    <xacro:aoba_joint name="rev21" can_interface="can2" motor_id="21" kp="30.0" kd="1.0" direction="-1"/>
+    <xacro:aoba_joint name="rev22" can_interface="can2" motor_id="22" kp="30.0" kd="1.0" direction="1"/>
+    <xacro:aoba_joint name="rev23" can_interface="can2" motor_id="23" kp="30.0" kd="1.0" direction="1"/>
+    <xacro:aoba_joint name="rev24" can_interface="can2" motor_id="24" kp="30.0" kd="1.0" direction="1"/>
+    <xacro:aoba_joint name="rev25" can_interface="can2" motor_id="25" kp="30.0" kd="1.0" direction="1"/>
   </ros2_control>
 </robot>
