Commit message: Add joint_state_bridge node and unify joint names to rev11 format
aoba_system.urdf.xacro のダミーモデルを廃止し aoba.xacro を include で取り込み、
ros2_control セクションと controllers.yaml のjoint名を rev11 形式に統一した。
/joint_states (11軸) → /forward_position_controller/commands (10軸) 変換を行う
ブリッジノードと、headless + bridge 構成の launch ファイルを追加。

Co-Authored-By: Claude Opus 4.6 (1M context) <noreply@anthropic.com>

File: ros2_ws/src/aoba_hardware/urdf/aoba_system.urdf.xacro (robot description, xacro)
@@ -17,20 +17,7 @@
   </xacro:macro>
   <!-- ================================================================== -->
-  <!-- Minimal robot description (dummy links for standalone testing)     -->
-  <!-- For the full model, use biped_description/urdf instead.            -->
+  <!-- Full robot model from aoba_description                             -->
   <!-- ================================================================== -->
-  <link name="base_link">
-    <visual>
-      <geometry>
-        <box size="0.1 0.1 0.1"/>
-      </geometry>
-    </visual>
-  </link>
-  <!-- Dummy link and fixed joint so URDF is valid with no movable joints -->
-  <link name="dummy_link"/>
-  <joint name="dummy_fixed" type="fixed">
-    <parent link="base_link"/>
-    <child link="dummy_link"/>
-  </joint>
+  <xacro:include filename="$(find aoba_description)/urdf/aoba.xacro"/>
   <!-- ================================================================== -->
   <!-- ros2_control configuration: 10 joints on 2 CAN buses              -->
@@ -41,15 +28,15 @@
     </hardware>
     <!-- Left leg (CAN1) -->
-    <xacro:aoba_joint name="left_hip_yaw_joint"     can_interface="can1" motor_id="11" kp="30.0" kd="1.0"/>
-    <xacro:aoba_joint name="left_hip_roll_joint"    can_interface="can1" motor_id="12" kp="30.0" kd="1.0"/>
-    <xacro:aoba_joint name="left_hip_pitch_joint"   can_interface="can1" motor_id="13" kp="30.0" kd="1.0"/>
-    <xacro:aoba_joint name="left_knee_pitch_joint"  can_interface="can1" motor_id="14" kp="30.0" kd="1.0"/>
-    <xacro:aoba_joint name="left_ankle_pitch_joint" can_interface="can1" motor_id="15" kp="30.0" kd="1.0"/>
+    <xacro:aoba_joint name="rev11" can_interface="can1" motor_id="11" kp="30.0" kd="1.0"/>
+    <xacro:aoba_joint name="rev12" can_interface="can1" motor_id="12" kp="30.0" kd="1.0"/>
+    <xacro:aoba_joint name="rev13" can_interface="can1" motor_id="13" kp="30.0" kd="1.0"/>
+    <xacro:aoba_joint name="rev14" can_interface="can1" motor_id="14" kp="30.0" kd="1.0"/>
+    <xacro:aoba_joint name="rev15" can_interface="can1" motor_id="15" kp="30.0" kd="1.0"/>
     <!-- Right leg (CAN2) -->
-    <xacro:aoba_joint name="right_hip_yaw_joint"     can_interface="can2" motor_id="21" kp="30.0" kd="1.0"/>
-    <xacro:aoba_joint name="right_hip_roll_joint"    can_interface="can2" motor_id="22" kp="30.0" kd="1.0"/>
-    <xacro:aoba_joint name="right_hip_pitch_joint"   can_interface="can2" motor_id="23" kp="30.0" kd="1.0"/>
-    <xacro:aoba_joint name="right_knee_pitch_joint"  can_interface="can2" motor_id="24" kp="30.0" kd="1.0"/>
-    <xacro:aoba_joint name="right_ankle_pitch_joint" can_interface="can2" motor_id="25" kp="30.0" kd="1.0"/>
+    <xacro:aoba_joint name="rev21" can_interface="can2" motor_id="21" kp="30.0" kd="1.0"/>
+    <xacro:aoba_joint name="rev22" can_interface="can2" motor_id="22" kp="30.0" kd="1.0"/>
+    <xacro:aoba_joint name="rev23" can_interface="can2" motor_id="23" kp="30.0" kd="1.0"/>
+    <xacro:aoba_joint name="rev24" can_interface="can2" motor_id="24" kp="30.0" kd="1.0"/>
+    <xacro:aoba_joint name="rev25" can_interface="can2" motor_id="25" kp="30.0" kd="1.0"/>
   </ros2_control>
 </robot>

Commit message: Feat/add sync rviz actual rs02 (#29)
* Move joint_limits.py to aoba_description and enable ament_cmake_python

joint_limits.py はロボット物理仕様に属するため aoba_description に移動し、
他パッケージから import 可能にするため ament_cmake_python を有効化した。
joint_gui.py の可動範囲ハードコードも joint_limits.py からの動的取得に変更。

Co-Authored-By: Claude Opus 4.6 (1M context) <noreply@anthropic.com>

* Add joint_state_bridge node and unify joint names to rev11 format

aoba_system.urdf.xacro のダミーモデルを廃止し aoba.xacro を include で取り込み、
ros2_control セクションと controllers.yaml のjoint名を rev11 形式に統一した。
/joint_states (11軸) → /forward_position_controller/commands (10軸) 変換を行う
ブリッジノードと、headless + bridge 構成の launch ファイルを追加。

Co-Authored-By: Claude Opus 4.6 (1M context) <noreply@anthropic.com>

* Allow partial motor activation with graceful probe degradation

on_activate() のプローブ失敗を ERROR から WARN に格下げし、
応答のないjointを disabled としてランタイムでスキップする。
モータ1個だけ接続してのテストが YAML 変更なしで可能になる。
全モータ未応答の場合のみ従来通り ERROR で停止。

Co-Authored-By: Claude Opus 4.6 (1M context) <noreply@anthropic.com>

* URDFで定めた回転方向と実際のモータの回転方向の符号を整合させるパラメータを追加

* Fix no ros2_control tag error by remapping robot_description topic

Jazzy (v4.x) の controller_manager は /robot_description トピックから
URDFを受信する仕様に変更されており、Mac側の robot_state_publisher が
ros2_controlタグなしのURDFを同トピックに配信すると衝突してクラッシュする。

全bringup launchで controller_manager の robot_description を
/hw/robot_description にリマップし、headless/with_bridge では
専用の robot_description_publisher ノードを追加して配信する構成にした。

また bringup_headless に joint_states_topic 引数を追加し、
配信先トピック名を起動時に選択可能にした。

Co-Authored-By: Claude Opus 4.6 (1M context) <noreply@anthropic.com>

* Separate trajectory command topic to /cmd/joint_states

trajectory_replay_node の配信先を /joint_states → /cmd/joint_states に変更し、
ハードウェア側の joint_state_broadcaster との競合を防止。
robot_state_publisher も /cmd/joint_states を購読するようリマップ。

また hw command を10軸に制限し、首関節(neck)を除外して
forward_position_controller の期待するサイズと一致させた。

Co-Authored-By: Claude Opus 4.6 (1M context) <noreply@anthropic.com>

* Enhance display_rviz_only.launch.py with topic remapping and PlotJuggler

joint_states_topic 引数を追加し、/cmd/joint_states 等の任意のトピックを
robot_state_publisher に接続可能にした。plot:=true で PlotJuggler を
同時起動できるようにし、RViz終了時に全プロセスを自動シャットダウンする
イベントハンドラを追加。

Co-Authored-By: Claude Opus 4.6 (1M context) <noreply@anthropic.com>

* Add RS02 motor fault/calibration diagnostic tool

CANソケットを通じてRS02モータにdisableコマンドを送信し、
type-2フィードバックフレームからフォルト状態・キャリブレーション状況・
温度等を一括確認するCLIツール。依存は標準ライブラリのみ。

Co-Authored-By: Claude Opus 4.6 (1M context) <noreply@anthropic.com>

* Update .claude session handover and settings

handover.md を現在の状態（bringup_headless正常動作確認済み）に更新。
settings.json に pixi install, pkill 等の許可パターンを追加。

Co-Authored-By: Claude Opus 4.6 (1M context) <noreply@anthropic.com>

* RS02対応: CANインターフェース名変更とモータ回転方向修正

URDFのCANインターフェースをcan1/can2からcan1_rs/can2_rsに変更し、
実機のネットワーク構成に合わせた。rev14, rev23, rev24, rev25の
回転方向符号を修正。bringup_headlessにjoint_statesの/hw/joint_states
へのリマップを追加。

Co-Authored-By: Claude Opus 4.6 (1M context) <noreply@anthropic.com>

* 軌道再生ノードに初期化ランプフェーズを追加

controlモードで起動時に/joint_statesから現在の関節角度を読み取り、
軌道の初期姿勢まで線形補間で滑らかに遷移する機能を追加。
状態機械(WAITING_FOR_STATE → MOVING_TO_INITIAL → REPLAYING)で管理。
各configにinit_duration/init_state_timeoutパラメータと歩行待機姿勢
(hip=-60deg, knee=90deg, ankle=-30deg)を設定。

Co-Authored-By: Claude Opus 4.6 (1M context) <noreply@anthropic.com>

* 歩行手順とRS02セットアップのドキュメント追加

how_to_walk_01.md: 歩行実験の手順書
setup_rs02.md: RS02モータのセットアップ手順書

Co-Authored-By: Claude Opus 4.6 (1M context) <noreply@anthropic.com>

* Claude Code許可設定を更新

CAN診断・udev・ROS2トピック関連のツール許可を追加。

Co-Authored-By: Claude Opus 4.6 (1M context) <noreply@anthropic.com>

* update process

---------

Co-authored-by: Claude Opus 4.6 (1M context) <noreply@anthropic.com>

File: ros2_ws/src/aoba_hardware/urdf/aoba_system.urdf.xacro (robot description, xacro)
@@ -4,5 +4,5 @@
   <!-- Xacro macro for a RobStride motor joint (ros2_control definition)  -->
   <!-- ================================================================== -->
-  <xacro:macro name="aoba_joint" params="name can_interface motor_id kp kd">
+  <xacro:macro name="aoba_joint" params="name can_interface motor_id kp kd direction">
     <joint name="${name}">
       <param name="can_interface">${can_interface}</param>
@@ -10,4 +10,5 @@
       <param name="kp">${kp}</param>
       <param name="kd">${kd}</param>
+      <param name="direction">${direction}</param>
       <command_interface name="position"/>
       <state_interface name="position"/>
@@ -17,20 +18,7 @@
   </xacro:macro>
   <!-- ================================================================== -->
-  <!-- Minimal robot description (dummy links for standalone testing)     -->
-  <!-- For the full model, use biped_description/urdf instead.            -->
+  <!-- Full robot model from aoba_description                             -->
   <!-- ================================================================== -->
-  <link name="base_link">
-    <visual>
-      <geometry>
-        <box size="0.1 0.1 0.1"/>
-      </geometry>
-    </visual>
-  </link>
-  <!-- Dummy link and fixed joint so URDF is valid with no movable joints -->
-  <link name="dummy_link"/>
-  <joint name="dummy_fixed" type="fixed">
-    <parent link="base_link"/>
-    <child link="dummy_link"/>
-  </joint>
+  <xacro:include filename="$(find aoba_description)/urdf/aoba.xacro"/>
   <!-- ================================================================== -->
   <!-- ros2_control configuration: 10 joints on 2 CAN buses              -->
@@ -41,15 +29,15 @@
     </hardware>
     <!-- Left leg (CAN1) -->
-    <xacro:aoba_joint name="left_hip_yaw_joint"     can_interface="can1" motor_id="11" kp="30.0" kd="1.0"/>
-    <xacro:aoba_joint name="left_hip_roll_joint"    can_interface="can1" motor_id="12" kp="30.0" kd="1.0"/>
-    <xacro:aoba_joint name="left_hip_pitch_joint"   can_interface="can1" motor_id="13" kp="30.0" kd="1.0"/>
-    <xacro:aoba_joint name="left_knee_pitch_joint"  can_interface="can1" motor_id="14" kp="30.0" kd="1.0"/>
-    <xacro:aoba_joint name="left_ankle_pitch_joint" can_interface="can1" motor_id="15" kp="30.0" kd="1.0"/>
+    <xacro:aoba_joint name="rev11" can_interface="can1_rs" motor_id="11" kp="30.0" kd="1.0" direction="-1"/>
+    <xacro:aoba_joint name="rev12" can_interface="can1_rs" motor_id="12" kp="30.0" kd="1.0" direction="1"/>
+    <xacro:aoba_joint name="rev13" can_interface="can1_rs" motor_id="13" kp="30.0" kd="1.0" direction="1"/>
+    <xacro:aoba_joint name="rev14" can_interface="can1_rs" motor_id="14" kp="30.0" kd="1.0" direction="-1"/>
+    <xacro:aoba_joint name="rev15" can_interface="can1_rs" motor_id="15" kp="30.0" kd="1.0" direction="1"/>
     <!-- Right leg (CAN2) -->
-    <xacro:aoba_joint name="right_hip_yaw_joint"     can_interface="can2" motor_id="21" kp="30.0" kd="1.0"/>
-    <xacro:aoba_joint name="right_hip_roll_joint"    can_interface="can2" motor_id="22" kp="30.0" kd="1.0"/>
-    <xacro:aoba_joint name="right_hip_pitch_joint"   can_interface="can2" motor_id="23" kp="30.0" kd="1.0"/>
-    <xacro:aoba_joint name="right_knee_pitch_joint"  can_interface="can2" motor_id="24" kp="30.0" kd="1.0"/>
-    <xacro:aoba_joint name="right_ankle_pitch_joint" can_interface="can2" motor_id="25" kp="30.0" kd="1.0"/>
+    <xacro:aoba_joint name="rev21" can_interface="can2_rs" motor_id="21" kp="30.0" kd="1.0" direction="-1"/>
+    <xacro:aoba_joint name="rev22" can_interface="can2_rs" motor_id="22" kp="30.0" kd="1.0" direction="1"/>
+    <xacro:aoba_joint name="rev23" can_interface="can2_rs" motor_id="23" kp="30.0" kd="1.0" direction="-1"/>
+    <xacro:aoba_joint name="rev24" can_interface="can2_rs" motor_id="24" kp="30.0" kd="1.0" direction="1"/>
+    <xacro:aoba_joint name="rev25" can_interface="can2_rs" motor_id="25" kp="30.0" kd="1.0" direction="-1"/>
   </ros2_control>
 </robot>
